File: pcb/crimpdeq/crimpdeq.kicad_sch (KiCad schematic)
At the start: 55 parts, among them J10 A-_Cable_Pad, J11 E+_Cable_Pad, J12 E-_Cable_Pad, J2 USB4105-GF-A, J5 B-_Cable_Pad, J6 SW+_Cable_Pad, J7 B+_Cable_Pad, J8 SW-_Cable_Pad, J9 A+_Cable_Pad, Q2 DMG3415U, U1 ESP32-C3-MINI-1, U2 MCP73831T-2ACI/OT, U3 ADS1220, U5 MAX17048G+T10, U6 SY8088

Commit message: fix: improve ADC bypassing and reconcile assembly metadata
Parts:
- R7, R8: LCSC C25741 -> C25076
Changed lines of the file:
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@@
 			)
 		)
-		(property "LCSC" "C25741"
+		(property "LCSC" "C25076"
 			(at 31.75 146.05 0)
 			(hide yes)
@@
 			)
 		)
-		(property "LCSC" "C25741"
+		(property "LCSC" "C25076"
 			(at 31.75 153.67 0)
 			(hide yes)

Commit message: fix: align prototype metadata and clean board annotations
Parts:
- C11, C19: footprint Capacitor_SMD:C_0603_1608Metric -> C_0603_1608Metric
- J10, J11, J12, J5, J6, J7, J8, J9: now not fitted
- U3: footprint Package_SO:TSSOP-16_4.4x5mm_P0.65mm -> TSSOP-16_4.4x5mm_P0.65mm
Connections:
- net Net-(U3-AIN0): now reaches C12.1, R7.1, U3.11 (AIN0/REFP1)
Changed lines of the file:
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@@
 		)
 	)
-	(label "Buck_Coil"
+	(global_label "Net-(U3-AIN0)"
+		(shape bidirectional)
+		(at 55.88 146.05 0)
+		(effects
+			(font
+				(size 1.27 1.27)
+			)
+			(justify left bottom)
+		)
+		(property "Intersheetrefs" "${INTERSHEET_REFS}"
+			(at 55.88 146.05 0)
+			(hide yes)
+			(show_name no)
+			(do_not_autoplace no)
+			(effects
+				(font
+					(size 1.27 1.27)
+				)
+			)
+		)
+	)
+	(global_label "Buck_Coil"
+		(shape bidirectional)
 		(at 236.22 73.66 0)
 		(effects
@@
 			(justify left bottom)
 		)
+		(property "Intersheetrefs" "${INTERSHEET_REFS}"
+			(at 236.22 73.66 0)
+			(hide yes)
+			(show_name no)
+			(do_not_autoplace no)
+			(effects
+				(font
+					(size 1.27 1.27)
+				)
+			)
+		)
 	)
 	(global_label "SW_BATT"
@@
 			)
 		)
-		(property "Datasheet" "https://www.diodes.com/assets/Datasheets/ds31785.pdf"
+		(property "Datasheet" "https://www.diodes.com/assets/Datasheets/DMG2301L.pdf"
 			(at 146.05 153.67 0)
 			(hide yes)
@@
 		(on_board yes)
 		(in_pos_files yes)
-		(dnp no)
+		(dnp yes)
 		(property "Reference" "J6"
 			(at 215.9 131.064 0)
@@
 		(on_board yes)
 		(in_pos_files yes)
-		(dnp no)
+		(dnp yes)
 		(property "Reference" "J10"
 			(at 241.3 114.554 0)
@@
 		(on_board yes)
 		(in_pos_files yes)
-		(dnp no)
+		(dnp yes)
 		(property "Reference" "J7"
 			(at 215.9 114.808 0)
@@
 		(on_board yes)
 		(in_pos_files yes)
-		(dnp no)
+		(dnp yes)
 		(property "Reference" "J5"
 			(at 215.646 107.696 0)
@@
 		(on_board yes)
 		(in_pos_files yes)
-		(dnp no)
+		(dnp yes)
 		(property "Reference" "J8"
 			(at 215.9 123.19 0)
@@
 			)
 		)
-		(property "Footprint" "Package_SO:TSSOP-16_4.4x5mm_P0.65mm"
+		(property "Footprint" "TSSOP-16_4.4x5mm_P0.65mm"
 			(at 82.55 142.24 0)
 			(hide yes)
@@
 		(on_board yes)
 		(in_pos_files yes)
-		(dnp no)
+		(dnp yes)
 		(property "Reference" "J11"
 			(at 241.3 121.666 0)
@@
 		(on_board yes)
 		(in_pos_files yes)
-		(dnp no)
+		(dnp yes)
 		(property "Reference" "J12"
 			(at 241.3 129.794 0)
@@
 		(on_board yes)
 		(in_pos_files yes)
-		(dnp no)
+		(dnp yes)
 		(property "Reference" "J9"
 			(at 241.3 108.204 0)
@@
 			)
 		)
-		(property "Footprint" "Capacitor_SMD:C_0603_1608Metric"
+		(property "Footprint" "C_0603_1608Metric"
 			(at 59.69 120.65 0)
 			(hide yes)
@@
 			)
 		)
-		(property "Footprint" "Capacitor_SMD:C_0603_1608Metric"
+		(property "Footprint" "C_0603_1608Metric"
 			(at 72.39 120.65 0)
 			(hide yes)
@@
 			)
 		)
-		(property "Datasheet" "https://datasheets.maximintegrated.com/en/ds/MAX17048-MAX17049.pdf"
+		(property "Datasheet" ""
 			(at 149.86 111.76 0)
 			(hide yes)
