File: pcb/crimpdeq/crimpdeq.kicad_pcb (KiCad board)
At the start: 4 copper layers, 30 x 30 mm, 55 parts, among them J10 A-_Cable_Pad, J11 E+_Cable_Pad, J12 E-_Cable_Pad, J2 USB4105-GF-A, J5 B-_Cable_Pad, J6 SW+_Cable_Pad, J7 B+_Cable_Pad, J8 SW-_Cable_Pad, J9 A+_Cable_Pad, Q2 DMG3415U, U1 ESP32-C3-MINI-1, U2 MCP73831T-2ACI/OT, U3 ADS1220, U5 MAX17048G+T10, U6 SY8088

Commit message: fix: remove vias from solder-paste apertures
Routing:
- net GND: track 189.0 -> 190.4 mm
- net VBUS: track 42.3 -> 41.7 mm, vias 3 -> 2
- net unconnected-(U1-NC-Pad10): track 0.34 -> 0.00 mm, vias 1 -> 0
Changed lines of the file:
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@@
 	)
 	(segment
+		(start 140.4 61.2)
+		(end 140 59.95)
+		(width 0.2)
+		(layer "F.Cu")
+		(net "GND")
+	)
+	(segment
 		(start 148.247 74.0468)
 		(end 150.663 74.0468)
@@
 	)
 	(segment
-		(start 132.475 63.025)
-		(end 134 61.5)
-		(width 0.2)
-		(layer "F.Cu")
-		(net "GND")
-	)
-	(segment
 		(start 154 70.75)
 		(end 154.4875 70.75)
@@
 	)
 	(segment
-		(start 140 60.8)
-		(end 140 59.95)
-		(width 0.2)
-		(layer "F.Cu")
-		(net "GND")
-	)
-	(segment
 		(start 135.949 54.3977)
 		(end 136.5 54.9486)
@@
 	)
 	(segment
+		(start 132.475 63.025)
+		(end 133.8 61.7)
+		(width 0.2)
+		(layer "F.Cu")
+		(net "GND")
+	)
+	(segment
 		(start 145.034 73.8341)
 		(end 143.8 75.0683)
@@
 	)
 	(via
-		(at 134 61.5)
-		(size 0.6)
-		(drill 0.3)
-		(layers "F.Cu" "B.Cu")
-		(locked yes)
-		(net "GND")
-	)
-	(via
 		(at 138 61.5)
 		(size 0.6)
@@
 	)
 	(via
-		(at 140 60.8)
+		(at 146.8 56.2)
 		(size 0.6)
 		(drill 0.3)
@@
 	)
 	(via
-		(at 146.8 56.2)
+		(at 145.8 54.2)
 		(size 0.6)
 		(drill 0.3)
@@
 	)
 	(via
-		(at 145.8 54.2)
+		(at 140.4 61.2)
 		(size 0.6)
 		(drill 0.3)
 		(layers "F.Cu" "B.Cu")
-		(locked yes)
 		(net "GND")
 	)
@@
 		(net "GND")
 	)
+	(via
+		(at 133.8 61.7)
+		(size 0.5)
+		(drill 0.3)
+		(layers "F.Cu" "B.Cu")
+		(net "GND")
+	)
 	(segment
 		(start 145 63.1)
@@
 	)
 	(segment
+		(start 140.4 61.2)
+		(end 139.3 61.5)
+		(width 0.2)
+		(layer "B.Cu")
+		(net "GND")
+	)
+	(segment
 		(start 128.39 64.8)
 		(end 128.39 61.8586)
@@
 	)
 	(segment
-		(start 134 61.5)
-		(end 134.1 61.4)
+		(start 147.75 63.15)
+		(end 147.75 62.4983)
 		(width 0.2)
 		(layer "B.Cu")
@@
 	)
 	(segment
-		(start 147.75 63.15)
-		(end 147.75 62.4983)
+		(start 146.8 62.3983)
+		(end 146.998 62.2)
 		(width 0.2)
 		(layer "B.Cu")
@@
 	)
 	(segment
-		(start 146.8 62.3983)
-		(end 146.998 62.2)
+		(start 140.4 61.2)
+		(end 139.825 60.625)
 		(width 0.2)
 		(layer "B.Cu")
@@
 	)
 	(segment
-		(start 140 60.8)
-		(end 139.825 60.625)
-		(width 0.2)
-		(layer "B.Cu")
-		(net "GND")
-	)
-	(segment
 		(start 141.8 58.2)
 		(end 143.775 58.2)
@@
 	)
 	(segment
+		(start 133.8 61.7)
+		(end 134.1 61.4)
+		(width 0.2)
+		(layer "B.Cu")
+		(net "GND")
+	)
+	(segment
 		(start 151.4 59.32)
 		(end 152.048 58.6715)
@@
 	)
 	(segment
-		(start 139.3 61.5)
-		(end 140 60.8)
-		(width 0.2)
-		(layer "B.Cu")
-		(net "GND")
-	)
-	(segment
-		(start 134 61.5)
-		(end 135.11 60.39)
-		(width 0.2)
-		(layer "In2.Cu")
-		(net "GND")
-	)
-	(segment
 		(start 139 69)
 		(end 137.614 67.6143)
@@
 	)
 	(segment
+		(start 133.8 61.7)
+		(end 135.11 60.39)
+		(width 0.2)
+		(layer "In2.Cu")
+		(net "GND")
+	)
+	(segment
 		(start 146.8 56.2)
 		(end 147 56)
@@
 	)
 	(via
-		(at 155 61.5)
-		(size 0.6)
-		(drill 0.3)
-		(layers "F.Cu" "B.Cu")
-		(net "VBUS")
-	)
-	(via
 		(at 148.22 67.4712)
 		(size 0.6)
@@
 	)
 	(segment
-		(start 155 62.05)
-		(end 155 61.5)
-		(width 0.2)
-		(layer "B.Cu")
-		(net "VBUS")
-	)
-	(segment
 		(start 134.088 59.425)
 		(end 132.45 61.0625)
@@
 		(net "Net-(U2-PROG)")
 	)
-	(via
-		(at 148 61.5)
-		(size 0.6)
-		(drill 0.3)
-		(layers "F.Cu" "B.Cu")
-		(locked yes)
-		(net "unconnected-(U1-NC-Pad10)")
-	)
-	(segment
-		(start 147.8 61.5)
-		(end 147.7 61.4)
-		(width 0.2)
-		(layer "B.Cu")
-		(net "unconnected-(U1-NC-Pad10)")
-	)
-	(segment
-		(start 148 61.5)
-		(end 147.8 61.5)
-		(width 0.2)
-		(layer "B.Cu")
-		(net "unconnected-(U1-NC-Pad10)")
-	)
 	(zone
